File: Kicad/NeotronF7.sch (KiCad schematic (older format))
At the start: 58 parts, among them J1 Conn_02x05_Odd_Even, J2 USB_B_Micro, J3 DB9_Male_MountingHoles, J4 ATAPI Interface 1, J5 SD_Card, J6 SD_Card, J7 ATAPI Interface 2, J8 Double-mini-DIN-6, U1 AMS1117-3.3, U2 STM32F767BGTx, U3 LY68S3200SLT, U5 MAX232, X1 50MHz XO, Y1 16 MHz, Y2 32.768 kHz

Commit message: Swap Flash for ESP-PSRAM as it's closer to the part we actually want.
Parts:
- removed U3: LY68S3200SLT, Package_SO:SOIC-8_3.9x4.9mm_P1.27mm, symbol Memory_Flash:AT25SF081-SSHD-X
- added U?: LY68S3200SLT, Package_SO:SOIC-8_3.9x4.9mm_P1.27mm, symbol Memory_RAM:ESP-PSRAM32
Connections:
- wire segments 390 -> 510
Other:
- note added: "TODO: This should now be MII, which\nmeans we can use a 25 MHz crystal"
- moved on the sheet: J8
