File: Kicad/Neotron-528ST.sch (KiCad schematic (older format))
At the start: 58 parts, among them J1 Conn_02x05_Odd_Even, J2 USB_B_Micro, J3 DB9_Male_MountingHoles, J4 ATAPI Interface 1, J5 SD_Card, J6 SD_Card, J7 ATAPI Interface 2, J8 Double-mini-DIN-6, U1 AMS1117-3.3, U101 LY68S3200SLT, U2 STM32F767BGTx, U5 MAX232, X1 50MHz XO, Y1 16 MHz, Y2 32.768 kHz

Commit message: Removed USB FS hub. Added stacked USB A connector.
Parts:
- added C108: 100n, Capacitor_SMD:C_0402_1005Metric, symbol Device:C
- C109: renamed from C1; footprint (none) -> Capacitor_SMD:C_0402_1005Metric
- C110: renamed from C6; footprint (none) -> Capacitor_SMD:C_0402_1005Metric
- C111: renamed from C17; footprint (none) -> Capacitor_SMD:C_0402_1005Metric
- C112: renamed from C16; footprint (none) -> Capacitor_SMD:C_0402_1005Metric
- J101: renamed from J2; value USB_B_Micro -> USB_B; footprint (none) -> Connector_USB:USB_B_OST_USB-B1HSxx_Horizontal; symbol Connector:USB_B_Micro -> Connector:USB_B
- R101: renamed from R3; footprint (none) -> Resistor_SMD:R_0402_1005Metric
- R102: renamed from R4; footprint (none) -> Resistor_SMD:R_0402_1005Metric
- R103: renamed from R5; footprint (none) -> Resistor_SMD:R_0402_1005Metric
- R104: renamed from R1; footprint (none) -> Resistor_SMD:R_0402_1005Metric
- R105: renamed from R2; footprint (none) -> Resistor_SMD:R_0402_1005Metric
- renumbered BT1 to BT101, C12 to C101, C14 to C102, C15 to C103, C31 to C104, C32 to C105, C11 to C106, C13 to C107, C2 to C113, C7 to C114, C3 to C115, C8 to C116, C4 to C117, C9 to C118, C18 to C119, C19 to C120, C21 to C121, C23 to C122, C25 to C123, C27 to C124, C29 to C125, C5 to C126, C10 to C127, C20 to C128, C22 to C129, C24 to C130, C26 to C131, C28 to C132, C30 to C133, F1 to F101, FB1 to FB101, FB3 to FB102, FB2 to FB103, J8 to J102, J1 to J103, J3 to J104, J4 to J105, J7 to J106, J5 to J107, J6 to J108, JP1 to JP101, U1 to U101, U101 to U102, U2 to U103, U5 to U104, X1 to X101, Y1 to Y101, Y2 to Y102
Connections:
- net labels added: LTDC_B[7..3], LTDC_G[7..2], LTDC_R[7..3]
- net labels removed: RCC_CLK_USB48, USB_OTG_HS_D+, USB_OTG_HS_D-, ~QUADSPI_BK1_CS
- wire segments 510 -> 513
- no-connect marks 7 -> 58
Other:
- moved on the sheet: FB103, U102
