File: Kicad/Neotron-500.sch (KiCad schematic (older format))
At the start: 59 parts, among them J101 USB_B, J102 Double-mini-DIN-6, J103 Conn_02x05_Odd_Even, J104 DB9_Male_MountingHoles, J105 ATAPI Interface 1, J106 ATAPI Interface 2, J107 SD_Card, J108 SD_Card, U101 AMS1117-3.3, U102 LY68S3200SLT, U103 STM32F767BGTx, U104 MAX232, X101 50MHz XO, Y101 16 MHz, Y102 32.768 kHz

Commit message: Swap to H7 in the Schematic
Parts:
- removed R102, R103: 0R, Resistor_SMD:R_0402_1005Metric, symbol Device:R
- removed U103: STM32F767BGTx, Package_QFP:LQFP-208_28x28mm_P0.5mm, symbol MCU_ST_STM32F7:STM32F767BGTx
- added U?: STM32H753IITx, Package_QFP:LQFP-176_24x24mm_P0.5mm, symbol MCU_ST_STM32H7:STM32H753IITx
Connections:
- net labels added: DEBUG_JTCK-SWCLK, DEBUG_JTMS-SWDIO, FMC_D10, FMC_D11, FMC_D12, FMC_D13, FMC_D14, FMC_D15, FMC_D8, FMC_D9, FMC_NBL0, FMC_NBL1, I2C1_SCL, I2C1_SDA, I2S2_SDI, I2S2_SDO, LTDC_B2, LTDC_R2, MDIOS_MDC, MDIOS_MDIO, QUADSPI_BK2_IO0, QUADSPI_BK2_IO1, QUADSPI_BK2_IO2, QUADSPI_BK2_IO3, QUADSPI_BK2_NCS, SDMMC2_CK, SDMMC2_CMD, SDMMC2_D0, SDMMC2_D1, SDMMC2_D2, SDMMC2_D3, SPI5_MISO, UART5_CTS, UART5_RTS, UART5_RX, UART5_TX, USB_OTG_FS_DM, USB_OTG_FS_DP, USB_OTG_HS_SOF
- net labels removed: RCC_MCO_1
- wire segments 513 -> 325
- no-connect marks 58 -> 6

Commit message: Schematic updates
Worked on USB Hub
Deleted QSPI SRAM
Added TSSOP-54 SDRAM (not wired up)
Parts:
- removed C108: 100n, Capacitor_SMD:C_0402_1005Metric, symbol Device:C
- removed U102: LY68S3200SLT, Package_SO:SOIC-8_3.9x4.9mm_P1.27mm, symbol Memory_RAM:ESP-PSRAM32
- added U105: W9864G6KH-6, TSOPII-54, symbol Memory_RAM:AS4C4M16SA
- J102: symbol ExtraConnectors:Double-mini-DIN-6 -> Neotron-500-rescue:Double-mini-DIN-6-ExtraConnectors
- U103: renamed from U?; value STM32H753IITx -> STM32H743IIT6
Connections:
- wire segments 325 -> 311
Other:
- note added: "System Design:\nSTM32H743IIT6 with VGA output via R2R DAC\nDP83848C 100base-T Ethernet PHY\nUSB3300 ULPI High-Speed PHY and USB2514 4-port Hub\nTLV320AIC23B I2S Audio Codec\nMAX232ESE RS-232 Driver\n\nTBD: 74HC245 bus transceiver and 74HC573 3-state Latch Parallel Port and ATA. Do we have room for the SRAM bus?\n"
- note removed: "System Design:\nSTM32F767IGT* with VGA output with 280 ohm R2R DAC\nTUSB2036 3-port USB 2.0 Full-speed Hub (12 Mbit/sec)\nDP83848C 100base-T Ethernet PHY\nTLV320AIC23B I2S Audio Codec*\nMAX232ESE RS-232 Driver\n74HC245 bus transceiver and 74HC573 3-state Latch Parallel Port and ATA\n\nNote that it's not possible to have an external USB 2.0 High-speed ULPI\nPHY, and the LCD-TFT output, AND the Eth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"
Changed lines of the file:
@@
 $Descr A2 23386 16535
 encoding utf-8
-Sheet 1 6
+Sheet 1 5
 Title "Neotron F7"
 Date "2020-05-25"
@@
 $EndComp
 Text Notes 16875 3475 0    100  Italic 0
-System Design:\nSTM32F767IGT* with VGA output with 280 ohm R2R DAC\nTUSB2036 3-port USB 2.0 Full-speed Hub (12 Mbit/sec)\nDP83848C 100base-T Ethernet PHY\nTLV320AIC23B I2S Audio Codec*\nMAX232ESE RS-232 Driver\n74HC245 bus transceiver and 74HC573 3-state Latch Parallel Port and ATA\n\nNote that it's not possible to have an external USB 2.0 High-speed ULPI\nPHY, and the LCD-TFT output, AND the Ethernet MAC. I concluded the\nEthernet MAC was more useful than 480 Mbps USB.
+System Design:\nSTM32H743IIT6 with VGA output via R2R DAC\nDP83848C 100base-T Ethernet PHY\nUSB3300 ULPI High-Speed PHY and USB2514 4-port Hub\nTLV320AIC23B I2S Audio Codec\nMAX232ESE RS-232 Driver\n\nTBD: 74HC245 bus transceiver and 74HC573 3-state Latch Parallel Port and ATA. Do we have room for the SRAM bus?\n
 $Comp
 L Interface_UART:MAX232 U104
@@
 USB Power Input - 2.5A max
 $Comp
-L ExtraConnectors:Double-mini-DIN-6 J102
+L Neotron-500-rescue:Double-mini-DIN-6-ExtraConnectors J102
 U 1 1 5EF144BD
 P 13025 4975
@@
 F11 "CRS_DV" O R 15382 7775 50
 F12 "ETH_REF_CLK" I L 14657 8025 50
-$EndSheet
-$Sheet
-S 17150 8875 700  850
-U 5EF25502
-F0 "IEEE1284 Parallel Port" 50
-F1 "ieee1284.sch" 50
 $EndSheet
 $Comp
@@
 Text Label -2325 8850 0    50   ~ 0
 FMC_A22
-Text Label 20075 6550 0    50   ~ 0
-QUADSPI_CLK
 Text Label -6375 6175 0    50   ~ 0
 ETH_MDC
@@
 Text Label -6375 6775 0    50   ~ 0
 ETH_TXD3
-Text Label 20075 6450 0    50   ~ 0
-QUADSPI_BK1_NCS
 Text Label -7700 6225 0    50   ~ 0
 USB_OTG_HS_ULPI_D7
@@
 Text Label -7700 6425 0    50   ~ 0
 USB_OTG_HS_ULPI_STP
-Text Label 20075 6850 0    50   ~ 0
-QUADSPI_BK1_IO1
-Text Label 20075 6950 0    50   ~ 0
-QUADSPI_BK1_IO0
-Text Label 20075 6750 0    50   ~ 0
-QUADSPI_BK1_IO2
-Text Label 20075 6650 0    50   ~ 0
-QUADSPI_BK1_IO3
 Text Label 13000 14925 0    50   ~ 0
 LTDC_VSYNC
@@
 Entry Wire Line
 	-1550 8950 -1450 9050
-$Comp
-L Memory_RAM:ESP-PSRAM32 U102
-U 1 1 6438446A
-P 21250 6750
-F 0 "U102" H 21050 7225 50  0000 R CNN
-F 1 "LY68S3200SLT" H 21825 7225 50  0000 R CNN
-F 2 "Package_SO:SOIC-8_3.9x4.9mm_P1.27mm" H 21250 6150 50  0001 C CNN
-F 3 "" H 20850 7250 50  0001 C CNN
-	1    21250 6750
-	-1   0    0    -1
-$EndComp
 $Sheet
 S 16500 4525 1875 1500
@@
 	0    -1   -1   0
 $EndComp
-$Comp
-L power:+3.3V #PWR0124
-U 1 1 61B2AC77
-P 21350 6100
-F 0 "#PWR0124" H 21350 5950 50  0001 C CNN
-F 1 "+3.3V" H 21365 6273 50  0000 C CNN
-F 2 "" H 21350 6100 50  0001 C CNN
-F 3 "" H 21350 6100 50  0001 C CNN
-	1    21350 6100
-	1    0    0    -1
-$EndComp
-$Comp
-L power:GND #PWR0125
-U 1 1 61B2C07F
-P 21350 7350
-F 0 "#PWR0125" H 21350 7100 50  0001 C CNN
-F 1 "GND" H 21355 7177 50  0000 C CNN
-F 2 "" H 21350 7350 50  0001 C CNN
-F 3 "" H 21350 7350 50  0001 C CNN
-	1    21350 7350
-	1    0    0    -1
-$EndComp
-$Comp
-L Device:C C108
-U 1 1 61B2CDF6
-P 21800 6650
-F 0 "C108" H 21915 6696 50  0000 L CNN
-F 1 "100n" H 21915 6605 50  0000 L CNN
-F 2 "Capacitor_SMD:C_0402_1005Metric" H 21838 6500 50  0001 C CNN
-F 3 "~" H 21800 6650 50  0001 C CNN
-	1    21800 6650
-	1    0    0    -1
-$EndComp
 Entry Bus Bus
 	13500 15025 13600 15125
@@
 	1675 5975 2050 5975
 Wire Wire Line
-	20025 6550 20850 6550
-Wire Wire Line
-	20025 6850 20850 6850
-Wire Wire Line
-	20025 6950 20850 6950
-Wire Wire Line
-	20025 6750 20850 6750
-Wire Wire Line
-	20025 6650 20850 6650
-Wire Wire Line
 	-2525 5850 -1700 5850
 Wire Wire Line
@@
 Wire Wire Line
 	-6425 6775 -5600 6775
-Wire Wire Line
-	20025 6450 20850 6450
 Wire Wire Line
 	-7750 6225 -6925 6225
@@
 Wire Wire Line
 	1425 2325 1425 2275
-Wire Wire Line
-	21350 6100 21350 6175
-Wire Wire Line
-	21350 7250 21350 7300
-Wire Wire Line
-	21350 7300 21800 7300
-Wire Wire Line
-	21800 7300 21800 6800
-Wire Wire Line
-	21800 6175 21350 6175
-Wire Wire Line
-	21800 6500 21800 6175
-Connection ~ 21350 7300
-Wire Wire Line
-	21350 7300 21350 7350
-Connection ~ 21350 6175
-Wire Wire Line
-	21350 6175 21350 6250
 Wire Bus Line
 	17125 15850 16350 15850
@@
 	3850 3175 3850 3300
 $Comp
-L MCU_ST_STM32H7:STM32H753IITx U?
+L MCU_ST_STM32H7:STM32H753IITx U103
 U 1 1 5EFD158A
 P 4650 7700
-F 0 "U?" H 5700 3350 50  0000 C CNN
-F 1 "STM32H753IITx" H 5700 3250 50  0000 C CNN
+F 0 "U103" H 5700 3350 50  0000 C CNN
+F 1 "STM32H743IIT6" H 5700 3250 50  0000 C CNN
 F 2 "Package_QFP:LQFP-176_24x24mm_P0.5mm" H 3450 3400 50  0001 R CNN
 F 3 "http://www.st.com/st-web-ui/static/active/en/resource/technical/document/datasheet/DM00388325.pdf" H 4650 7700 50  0001 C CNN
@@
 Wire Wire Line
 	3175 2400 5000 2400
+$Comp
+L Memory_RAM:AS4C4M16SA U105
+U 1 1 5F954597
+P 19750 12025
+F 0 "U105" H 19750 13506 50  0000 C CNN
+F 1 "W9864G6KH-6" H 19750 13415 50  0000 C CNN
+F 2 "TSOPII-54" H 19750 12025 50  0001 C CIN
+F 3 "https://www.alliancememory.com/wp-content/uploads/pdf/dram/64M-AS4C4M16SA-CI_v3.0_March%202015.pdf" H 19750 11775 50  0001 C CNN
+	1    19750 12025
+	1    0    0    -1
+$EndComp
 $EndSCHEMATC

Commit message: Tidying up schematic, and README.
Parts:
- removed BT101: 3V RTC Backup, symbol Device:Battery_Cell
- removed C101, C103, C105: 22u, Capacitor_SMD:C_0805_2012Metric, symbol Device:CP
- removed C102, C104, C113, C115, C117, C119, C120, C121, C122, C123, C124, C125, C126, C128, C129, C130, C131, C132, C133: 100n, Capacitor_SMD:C_0402_1005Metric, symbol Device:C
- removed C106, C107: 2.2u, Capacitor_SMD:C_0805_2012Metric, symbol Device:C
- removed C109, C110, C111, C112: 9p, Capacitor_SMD:C_0402_1005Metric, symbol Device:C
- removed C114, C116, C118, C127: 1u, Capacitor_SMD:C_0402_1005Metric, symbol Device:C
- removed F101: 2.5A, Capacitor_THT:C_Disc_D9.0mm_W2.5mm_P5.00mm, symbol Device:Polyfuse
- removed FB101, FB102, FB103: 100R@100MHz, Inductor_SMD:L_0805_2012Metric, symbol Device:Ferrite_Bead
- removed J101: USB_B, Connector_USB:USB_B_OST_USB-B1HSxx_Horizontal, symbol Connector:USB_B
- removed J102: Double-mini-DIN-6, symbol Neotron-500-rescue:Double-mini-DIN-6-ExtraConnectors
- removed J103: Conn_02x05_Odd_Even, symbol Connector_Generic:Conn_02x05_Odd_Even
- removed J104: DB9_Male_MountingHoles, symbol Connector:DB9_Male_MountingHoles
- removed J105: ATAPI Interface 1, symbol Connector_Generic:Conn_02x20_Odd_Even
- removed J106: ATAPI Interface 2, symbol Connector_Generic:Conn_02x20_Odd_Even
- removed J107, J108: SD_Card, symbol Connector:SD_Card
- removed JP101: Boot Mode Select, symbol Device:Jumper_NC_Dual
- removed R101: 0R, Resistor_SMD:R_0402_1005Metric, symbol Device:R
- removed R104, R105: 10k, Resistor_SMD:R_0402_1005Metric, symbol Device:R
- removed U101: AMS1117-3.3, Package_TO_SOT_SMD:SOT-223-3_TabPin2, symbol Regulator_Linear:AMS1117-3.3
- removed U103: STM32H743IIT6, Package_QFP:LQFP-176_24x24mm_P0.5mm, symbol MCU_ST_STM32H7:STM32H753IITx
- removed U104: MAX232, Package_SO:SOIC-16_3.9x9.9mm_P1.27mm, symbol Interface_UART:MAX232
- removed U105: W9864G6KH-6, TSOPII-54, symbol Memory_RAM:AS4C4M16SA
- removed X101: 50MHz XO, Oscillator:Oscillator_SMD_TXC_7C-4Pin_5.0x3.2mm, symbol Oscillator:TXC-7C
- removed Y101: 16 MHz, symbol Device:Crystal
- removed Y102: 32.768 kHz, symbol Device:Crystal
Connections:
- net labels removed: +3.3V, +5V, +BATT, DEBUG_JTCK-SWCLK, DEBUG_JTMS-SWDIO, ETH_COL, ETH_CRS, ETH_CRS_DV, ETH_MDC, ETH_MDIO, ETH_REF_CLK, ETH_RXD0, ETH_RXD1, ETH_RXD2, ETH_RXD3, ETH_RX_CLK, ETH_RX_DV, ETH_TDX0, ETH_TXD0, ETH_TXD1, ETH_TXD2, ETH_TXD3, ETH_TX_CLK, ETH_TX_EN, FMC_A0, FMC_A1, FMC_A10, FMC_A11, FMC_A12, FMC_A13, FMC_A14, FMC_A15, FMC_A16, FMC_A17, FMC_A18, FMC_A19, FMC_A2, FMC_A20, FMC_A21, FMC_A22, FMC_A23, FMC_A3, FMC_A4, FMC_A5, FMC_A6, FMC_A7, FMC_A8, FMC_A9, FMC_D0, FMC_D1, FMC_D10, FMC_D11, FMC_D12, FMC_D13, FMC_D14, FMC_D15, FMC_D2, FMC_D3, FMC_D4, FMC_D5, FMC_D6, FMC_D7, FMC_D8, FMC_D9, FMC_NBL0, FMC_NBL1, FMC_NE1, FMC_NOE, FMC_NWAIT, FMC_NWE, GND, I2C1_SCL, I2C1_SDA, I2C4_SCL, I2C4_SDA, I2S2_CK, I2S2_MCK, I2S2_SD, I2S2_SDI, I2S2_SDO, I2S2_WS, I2S3_CK, I2S3_SD, I2S3_WS, LTDC_B2, LTDC_B3, LTDC_B4, LTDC_B5, LTDC_B6, LTDC_B7, LTDC_B[7..3], LTDC_CLK, LTDC_DE, LTDC_G2, LTDC_G3, LTDC_G4, LTDC_G5, LTDC_G6, LTDC_G7, LTDC_G[7..2], LTDC_HSYNC, LTDC_R2, LTDC_R3, LTDC_R4, LTDC_R5, LTDC_R6, LTDC_R7, LTDC_R[7..3], LTDC_VSYNC, MDIOS_MDC, MDIOS_MDIO, QUADSPI_BK1_IO0, QUADSPI_BK1_IO1, QUADSPI_BK1_IO2, QUADSPI_BK1_IO3, QUADSPI_BK1_NCS, QUADSPI_BK2_IO0, QUADSPI_BK2_IO1, QUADSPI_BK2_IO2, QUADSPI_BK2_IO3, QUADSPI_BK2_NCS, QUADSPI_CLK, RCC_OSC32_IN, RCC_OSC32_OUT, RCC_OSC_IN, RCC_OSC_OUT, SDMMC1_CK, SDMMC1_CMD, SDMMC1_D0, SDMMC1_D1, SDMMC1_D2, SDMMC1_D3, SDMMC2_CK, SDMMC2_CMD, SDMMC2_D0, SDMMC2_D1, SDMMC2_D2, SDMMC2_D3, SPI4_MISO, SPI4_MOSI, SPI4_SCK, SPI5_MISO, SWDCLK, SWDIO, SWO, UART4_CTS, UART4_RTS, UART4_RX, UART4_TX, UART5_CTS, UART5_RTS, UART5_RX, UART5_TX, USART3_RX, USART3_TX, USB_OTG_FS_DM, USB_OTG_FS_DP, USB_OTG_HS_SOF, USB_OTG_HS_ULPI_CK, USB_OTG_HS_ULPI_D0, USB_OTG_HS_ULPI_D1, USB_OTG_HS_ULPI_D2, USB_OTG_HS_ULPI_D3, USB_OTG_HS_ULPI_D4, USB_OTG_HS_ULPI_D5, USB_OTG_HS_ULPI_D6, USB_OTG_HS_ULPI_D7, USB_OTG_HS_ULPI_DIR, USB_OTG_HS_ULPI_NXT, USB_OTG_HS_ULPI_STP, VDDA, VDD_MCU, VDD_SDMMC, VDD_USB, VREF+, ~RESET
- wire segments 311 -> 7
- no-connect marks 6 -> 1
Other:
- note removed: "Cortex-Debug"
- note removed: "Decoupling. Place one near to each power pin."
- note removed: "System Design:\nSTM32H743IIT6 with VGA output via R2R DAC\nDP83848C 100base-T Ethernet PHY\nUSB3300 ULPI High-Speed PHY and USB2514 4-port Hub\nTLV320AIC23B I2S Audio Codec\nMAX232ESE RS-232 Driver\n\nTBD: 74HC245 bus transceiver and 74HC573 3-state Latch Parallel Port and ATA. Do we have room for the SRAM bus?\n"
- note removed: "TODO: This should now be MII, which\nmeans we can use a 25 MHz crystal"
- note removed: "USB Power Input - 2.5A max"
